File: arduino_Uno_RevG-MU.sch (EAGLE design)
At the start: 48 parts, among them IC3 ADC, U4 ARDUINOR3-DIMENSION

Commit message: updated
Parts:
- removed U$33: CS, LS_ELECTRIC:1X2_HEADER1X2
- added U$14, U$15, U$16, U$17, U$20: 1X2_HEADER1X2, LS_ELECTRIC:1X2_HEADER1X2
- U$1, U$34, U$35, U$36: device LS_ELECTRIC:BNCBNC -> LS_ELECTRIC:BNC_INVBNC_INVERT
Connections:
- removed net IO6: U4.D6
- new net N$4: U$20.2, U$40.P$4
- new net N$5: U$20.1, U$40.P$5
- new net SS0: U$14.1, U4.D10(SS)
- new net SS1: U$15.1, U4.D8
- new net SS2: U$16.1, U4.D7
- new net SS3: U$17.1, U4.D6
- net CS3: no longer U$33.1
- net CS4: no longer U$33.2
- net IO4: now also U$40.P$2; no longer U$40.P$4
- net IO5: now also U$40.P$1; no longer U$40.P$5
- net RX: no longer U$40.P$1
- net SS: now also U$14.2, U$15.2, U$16.2, U$17.2; no longer U4.D10(SS)
- net TX: no longer U$40.P$2
Other:
- note removed: "RX"
- note removed: "TX"

Commit message: First board order
Connections:
- net 24GND renamed P_GND
- net 24VDC renamed PWR
Changed lines of the file:
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@@
-</segment>
-</net>
-<net name="24GND" class="0">
-<segment>
-<pinref part="OP1" gate="G$1" pin="C"/>
-<pinref part="C22" gate="G$1" pin="B"/>
-<wire x1="-63.5" y1="58.42" x2="-63.5" y2="45.72" width="0.1524" layer="91"/>
-<wire x1="-63.5" y1="45.72" x2="-81.28" y2="45.72" width="0.1524" layer="91"/>
-<wire x1="-81.28" y1="45.72" x2="-99.06" y2="45.72" width="0.1524" layer="91"/>
-<junction x="-81.28" y="45.72"/>
-<label x="-99.06" y="45.72" size="1.778" layer="95" rot="R180" xref="yes"/>
-</segment>
-<segment>
-<pinref part="U$40" gate="G$1" pin="P$8"/>
-<wire x1="-373.38" y1="233.68" x2="-363.22" y2="233.68" width="0.1524" layer="91"/>
-<label x="-363.22" y="233.68" size="1.778" layer="95" xref="yes"/>
-</segment>
-</net>
-<net name="24VDC" class="0">
-<segment>
-<pinref part="R13" gate="G$1" pin="A"/>
-<wire x1="-71.12" y1="106.68" x2="-71.12" y2="109.22" width="0.1524" layer="91"/>
-<wire x1="-71.12" y1="109.22" x2="-109.22" y2="109.22" width="0.1524" layer="91"/>
-<label x="-109.22" y="109.22" size="1.778" layer="95" rot="R180" xref="yes"/>
-</segment>
-<segment>
-<pinref part="U$40" gate="G$1" pin="P$10"/>
-<wire x1="-373.38" y1="243.84" x2="-363.22" y2="243.84" width="0.1524" layer="91"/>
-<label x="-363.22" y="243.84" size="1.778" layer="95" xref="yes"/>
 </segment>
 </net>
@@
 </segment>
 </net>
+<net name="PWR" class="0">
+<segment>
+<pinref part="R13" gate="G$1" pin="A"/>
+<wire x1="-71.12" y1="106.68" x2="-71.12" y2="109.22" width="0.1524" layer="91"/>
+<wire x1="-71.12" y1="109.22" x2="-109.22" y2="109.22" width="0.1524" layer="91"/>
+<label x="-109.22" y="109.22" size="1.778" layer="95" rot="R180" xref="yes"/>
+</segment>
+<segment>
+<pinref part="U$40" gate="G$1" pin="P$10"/>
+<wire x1="-373.38" y1="243.84" x2="-363.22" y2="243.84" width="0.1524" layer="91"/>
+<label x="-363.22" y="243.84" size="1.778" layer="95" xref="yes"/>
+</segment>
+</net>
+<net name="P_GND" class="0">
+<segment>
+<pinref part="OP1" gate="G$1" pin="C"/>
+<pinref part="C22" gate="G$1" pin="B"/>
+<wire x1="-63.5" y1="58.42" x2="-63.5" y2="45.72" width="0.1524" layer="91"/>
+<wire x1="-63.5" y1="45.72" x2="-81.28" y2="45.72" width="0.1524" layer="91"/>
+<wire x1="-81.28" y1="45.72" x2="-99.06" y2="45.72" width="0.1524" layer="91"/>
+<junction x="-81.28" y="45.72"/>
+<label x="-99.06" y="45.72" size="1.778" layer="95" rot="R180" xref="yes"/>
+</segment>
+<segment>
+<pinref part="U$40" gate="G$1" pin="P$8"/>
+<wire x1="-373.38" y1="233.68" x2="-363.22" y2="233.68" width="0.1524" layer="91"/>
+<label x="-363.22" y="233.68" size="1.778" layer="95" xref="yes"/>
+</segment>
+</net>
